File: pcb/display.kicad_sch (KiCad schematic)
At the start: 0 parts

Commit message: stuff
Parts:
- added C25, C27: 100nF, symbol Device:C_Small
- added C26: 1uF, symbol Device:C_Small
- added DS1: (no value), symbol DH03:LS013B7DH03
Connections:
- new net +3V3: C26.1, C27.1, DS1.6 (VDDA), DS1.7 (VDD), DS1.8 (EXTMODE)
- new net GND: C25.2, C26.2, C27.2, DS1.10 (VSSA), DS1.9 (VSS)
- new net P1.10: DS1.1 (SCLK)
- new net P1.11: DS1.2 (SI)
- new net P1.12: DS1.3 (SCS)
- new net P1.13: DS1.4 (EXTCOMIN)
- new net P1.14: C25.1, DS1.5 (DISP)

Commit message: sus commit
Parts:
- C25, C27: footprint (none) -> Capacitor_SMD:C_0402_1005Metric; LCSC Part (none) -> C1525
- C26: footprint (none) -> Capacitor_SMD:C_0402_1005Metric; LCSC Part (none) -> C52923
- DS1: LCSC Part (none) -> C127355
Changed lines of the file:
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@@
 			)
 		)
-		(property "Footprint" ""
+		(property "Footprint" "Capacitor_SMD:C_0402_1005Metric"
 			(at 177.8 82.55 0)
 			(hide yes)
@@
 		)
 		(property "Description" "Unpolarized capacitor, small symbol"
+			(at 177.8 82.55 0)
+			(hide yes)
+			(show_name no)
+			(do_not_autoplace no)
+			(effects
+				(font
+					(size 1.27 1.27)
+				)
+			)
+		)
+		(property "LCSC Part" "C1525"
 			(at 177.8 82.55 0)
 			(hide yes)
@@
 		)
 		(property "Description" ""
+			(at 148.59 81.28 0)
+			(hide yes)
+			(show_name no)
+			(do_not_autoplace no)
+			(effects
+				(font
+					(size 1.27 1.27)
+				)
+			)
+		)
+		(property "LCSC Part" "C127355"
 			(at 148.59 81.28 0)
 			(hide yes)
@@
 			)
 		)
-		(property "Footprint" ""
+		(property "Footprint" "Capacitor_SMD:C_0402_1005Metric"
 			(at 120.65 95.25 0)
 			(hide yes)
@@
 		)
 		(property "Description" "Unpolarized capacitor, small symbol"
+			(at 120.65 95.25 0)
+			(hide yes)
+			(show_name no)
+			(do_not_autoplace no)
+			(effects
+				(font
+					(size 1.27 1.27)
+				)
+			)
+		)
+		(property "LCSC Part" "C1525"
 			(at 120.65 95.25 0)
 			(hide yes)
@@
 			)
 		)
-		(property "Footprint" ""
+		(property "Footprint" "Capacitor_SMD:C_0402_1005Metric"
 			(at 173.99 82.55 0)
 			(hide yes)
@@
 			(at 173.99 82.55 0)
 			(hide yes)
+			(show_name no)
+			(do_not_autoplace no)
+			(effects
+				(font
+					(size 1.27 1.27)
+				)
+			)
+		)
+		(property "LCSC Part" "C52923"
+			(at 173.99 82.55 0)
+			(hide yes)

Commit message: sussy
Parts:
- DS1: footprint (none) -> JLCImport:5034801000
Connections:
- net +3V3: now also DS1.3 (EXTMODE), DS1.4 (VDD), DS1.5 (VDDA); no longer DS1.6 (VDDA), DS1.7 (VDD), DS1.8 (EXTMODE)
- net GND: now also DS1.1 (VSSA), DS1.2 (VSS); no longer DS1.10 (VSSA), DS1.9 (VSS)
- net P1.10: now also DS1.10 (SCLK); no longer DS1.1 (SCLK)
- net P1.11: now also DS1.9 (SI); no longer DS1.2 (SI)
- net P1.12: now also DS1.8 (SCS); no longer DS1.3 (SCS)
- net P1.13: now also DS1.7 (EXTCOMIN); no longer DS1.4 (EXTCOMIN)
- net P1.14: now also DS1.6 (DISP); no longer DS1.5 (DISP)
Other:
- note added: "TODO: Validate FPC before ordering this!!"
Changed lines of the file:
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@@
 	(generator_version "10.0")
 	(paper "A4")
+	(text "TODO: Validate FPC before ordering this!!\n"
+		(exclude_from_sim no)
+		(at 147.32 67.31 0)
+		(effects
+			(font
+				(size 1.27 1.27)
+			)
+		)
+	)
 	(junction
 		(at 153.67 80.01)
@@
 		(dnp no)
 		(fields_autoplaced yes)
-		(property "Reference" "#PWR042"
+		(property "Reference" "#PWR052"
 			(at 153.67 83.82 0)
 			(hide yes)
@@
 			(project "watch"
 				(path "/1ea987a7-f4cb-45bc-8f81-16ca70afed15"
-					(reference "#PWR042")
+					(reference "#PWR052")
 					(unit 1)
 				)
@@
 		(dnp no)
 		(fields_autoplaced yes)
-		(property "Reference" "#PWR045"
+		(property "Reference" "#PWR050"
 			(at 124.46 91.44 0)
 			(hide yes)
@@
 			(project "watch"
 				(path "/1ea987a7-f4cb-45bc-8f81-16ca70afed15"
-					(reference "#PWR045")
+					(reference "#PWR050")
 					(unit 1)
 				)
@@
 		(dnp no)
 		(fields_autoplaced yes)
-		(property "Reference" "#PWR043"
+		(property "Reference" "#PWR051"
 			(at 148.59 111.76 0)
 			(hide yes)
@@
 			(project "watch"
 				(path "/1ea987a7-f4cb-45bc-8f81-16ca70afed15"
-					(reference "#PWR043")
+					(reference "#PWR051")
 					(unit 1)
 				)
@@
 			)
 		)
-		(property "Footprint" ""
+		(property "Footprint" "JLCImport:5034801000"
 			(at 148.59 81.28 0)
 			(hide yes)
@@
 		(dnp no)
 		(fields_autoplaced yes)
-		(property "Reference" "#PWR044"
+		(property "Reference" "#PWR049"
 			(at 120.65 104.14 0)
 			(hide yes)
@@
 			(project "watch"
 				(path "/1ea987a7-f4cb-45bc-8f81-16ca70afed15"
-					(reference "#PWR044")
+					(reference "#PWR049")
 					(unit 1)
 				)
@@
 		(in_pos_files yes)
 		(dnp no)
-		(property "Reference" "#PWR046"
+		(property "Reference" "#PWR053"
 			(at 177.8 91.44 0)
 			(hide yes)
@@
 			(project "watch"
 				(path "/1ea987a7-f4cb-45bc-8f81-16ca70afed15"
-					(reference "#PWR046")
+					(reference "#PWR053")
 					(unit 1)
 				)

Commit message: mogus
Connections:
- net P1.10 renamed P1.01
- net P1.11 renamed P1.02
- net P1.12 renamed P1.04
- net P1.13 renamed P1.06
- net P1.14 renamed P1.07
Changed lines of the file:
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@@
 		)
 	)
-	(global_label "P1.12"
+	(global_label "P1.07"
 		(shape input)
-		(at 163.83 95.25 0)
+		(at 118.11 90.17 180)
 		(fields_autoplaced yes)
 		(effects
@@
 				(size 1.27 1.27)
 			)
-			(justify left)
+			(justify right)
 		)
 		(property "Intersheetrefs" "${INTERSHEET_REFS}"
-			(at 172.3185 95.25 0)
+			(at 109.6215 90.17 0)
 			(hide yes)
 			(show_name no)
@@
 					(size 1.27 1.27)
 				)
-				(justify left)
+				(justify right)
 			)
 		)
 	)
-	(global_label "P1.11"
+	(global_label "P1.06"
+		(shape input)
+		(at 134.62 92.71 180)
+		(fields_autoplaced yes)
+		(effects
+			(font
+				(size 1.27 1.27)
+			)
+			(justify right)
+		)
+		(property "Intersheetrefs" "${INTERSHEET_REFS}"
+			(at 126.1315 92.71 0)
+			(hide yes)
+			(show_name no)
+			(do_not_autoplace no)
+			(effects
+				(font
+					(size 1.27 1.27)
+				)
+				(justify right)
+			)
+		)
+	)
+	(global_label "P1.02"
 		(shape input)
 		(at 163.83 92.71 0)
@@
 		)
 	)
-	(global_label "P1.14"
-		(shape input)
-		(at 118.11 90.17 180)
-		(fields_autoplaced yes)
-		(effects
-			(font
-				(size 1.27 1.27)
-			)
-			(justify right)
-		)
-		(property "Intersheetrefs" "${INTERSHEET_REFS}"
-			(at 109.6215 90.17 0)
-			(hide yes)
-			(show_name no)
-			(do_not_autoplace no)
-			(effects
-				(font
-					(size 1.27 1.27)
-				)
-				(justify right)
-			)
-		)
-	)
-	(global_label "P1.13"
-		(shape input)
-		(at 134.62 92.71 180)
-		(fields_autoplaced yes)
-		(effects
-			(font
-				(size 1.27 1.27)
-			)
-			(justify right)
-		)
-		(property "Intersheetrefs" "${INTERSHEET_REFS}"
-			(at 126.1315 92.71 0)
-			(hide yes)
-			(show_name no)
-			(do_not_autoplace no)
-			(effects
-				(font
-					(size 1.27 1.27)
-				)
-				(justify right)
-			)
-		)
-	)
-	(global_label "P1.10"
+	(global_label "P1.01"
 		(shape input)
 		(at 163.83 90.17 0)
@@
 			(hide yes)
 			(show_name no)
+			(do_not_autoplace no)
+			(effects
+				(font
+					(size 1.27 1.27)
+				)
+				(justify left)
+			)
+		)
+	)
+	(global_label "P1.04"
+		(shape input)
+		(at 163.83 95.25 0)
+		(fields_autoplaced yes)
+		(effects
+			(font
+				(size 1.27 1.27)
+			)
+			(justify left)
+		)
+		(property "Intersheetrefs" "${INTERSHEET_REFS}"
+			(at 172.3185 95.25 0)
+			(hide yes)
+			(show_name no)
