File: pcb/pwr.kicad_sch (KiCad schematic)
At the start: 34 parts, among them J2 Adafruit Wireless Chg Module, SW6 PWR, U4 TPS63802DLAR, U5 TPS7A20xxxDQN, U6 BQ24074RGT, U7 MCP73831-2-OT, U9 TPS2116DRL

Commit message: starting le leyout
Parts:
- BT1: value Battery_Cell -> LiPo
- SW6: now not fitted; now left out of the parts list
Connections:
- net at BT1.1 (+): now also C22.1, U6.2 (BAT), U6.3 (BAT); no longer SW6.2 (B)
- removed net VBAT_RAW: C22.1, SW6.1 (A), U6.2 (BAT), U6.3 (BAT)
Other:
- moved on the sheet: C22

Commit message: mogus
Connections:
- net P1.05 is gone; now on net P1.15: U6.6 (EN1)
- net P1.15: no longer R17.2, U9.8 (ST)
- net P0.26: no longer names the net of U5.3 (EN)
- net P1.04 renamed P1.11
- net P1.06 renamed P1.10
- new net P1.13: R17.2, U9.8 (ST)
Other:
- note added: "INSERT NEW GPIO"
Changed lines of the file:
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@@
 	(generator_version "10.0")
 	(paper "A4")
+	(text "INSERT NEW GPIO\n"
+		(exclude_from_sim no)
+		(at 81.28 149.86 0)
+		(effects
+			(font
+				(size 1.27 1.27)
+			)
+		)
+	)
 	(junction
 		(at 97.79 88.9)
@@
 		)
 	)
-	(global_label "P1.04"
+	(global_label "P1.11"
 		(shape input)
 		(at 218.44 73.66 180)
@@
 		)
 	)
-	(global_label "P1.15"
+	(global_label "P1.13"
 		(shape input)
 		(at 173.99 50.8 0)
@@
 		)
 	)
-	(global_label "P0.26"
-		(shape input)
-		(at 86.36 149.86 180)
-		(fields_autoplaced yes)
-		(effects
-			(font
-				(size 1.27 1.27)
-			)
-			(justify right)
-		)
-		(property "Intersheetrefs" "${INTERSHEET_REFS}"
-			(at 77.8715 149.86 0)
-			(hide yes)
-			(show_name no)
-			(do_not_autoplace no)
-			(effects
-				(font
-					(size 1.27 1.27)
-				)
-				(justify right)
-			)
-		)
-	)
-	(global_label "P1.05"
+	(global_label "P1.15"
 		(shape input)
 		(at 218.44 78.74 180)
@@
 		)
 	)
-	(global_label "P1.06"
+	(global_label "P1.10"
 		(shape input)
 		(at 218.44 81.28 180)
