File: pcb/watch.kicad_pcb (KiCad board)
At the start: 6 copper layers, 47.2 x 35.5 mm, 61 parts, among them J1 USB_C_Receptacle_USB2.0_14P, J2 Adafruit Wireless Chg Module, U1 nRF52840, U2 USBLC6-2SC6, U3 MAX-M10S, U4 TPS63802DLAR, U5 TPS7A20xxxDQN, U6 BQ24074RGT, U8 RV-3028-C7, U9 TPS2116DRL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

Commit message: almost done?
Connections:
- E1 pad 2: (no net) -> GND
- E1 pad 3: (no net) -> GND
- E1 pad 4: (no net) -> GND
- E1 pad 5: (no net) -> GND
- E1 pad 6: (no net) -> GND
- E1 pad 7: (no net) -> GND
- E1 pad 8: (no net) -> GND
- E1 pad 9: (no net) -> GND
Routing:
- net GND: track 22.0 -> 27.2 mm, vias 8 -> 464
- net Net-(U3-RF_IN): track 3.66 -> 2.91 mm

Commit message: SUS!!
Routing:
- net GND: vias 464 -> 468
Changed lines of the file:
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@@
 		)
 		(embedded_fonts no)
-		(model "${KICAD10_3DMODEL_DIR}/RF_GPS.3dshapes/ublox_MAX.step"
+		(model "${KIPRJMOD}/libraries/MAX-M10S/MAX-M10S-00B.step"
 			(offset
 				(xyz 0 0 0)
@@
 			)
 			(rotate
-				(xyz 0 0 0)
+				(xyz -90 -0 -0)
 			)
 		)
@@
 		)
 		(embedded_fonts no)
-		(model "${KICAD10_3DMODEL_DIR}/Connector_JST.3dshapes/JST_PH_S2B-PH-SM4-TB_1x02-1MP_P2.00mm_Horizontal.step"
+		(model "${KICAD10_3DMODEL_DIR}/Connector_JST.3dshapes/JST_PH_S2B-PH-K_1x02_P2.00mm_Horizontal.step"
 			(offset
-				(xyz 0 0 0)
+				(xyz -1 1.5 0)
 			)
 			(scale
-				(xyz 1 1 1)
+				(xyz 1.2 1 1)
 			)
 			(rotate
-				(xyz 0 0 0)
+				(xyz -0 -0 -0)
 			)
 		)
@@
 		)
 		(embedded_fonts no)
-		(model "${KICAD10_3DMODEL_DIR}/Connector_USB.3dshapes/USB_C_Receptacle_G-Switch_GT-USB-7010ASV.step"
+		(model "${KICAD10_3DMODEL_DIR}/Connector_USB.3dshapes/USB_C_Receptacle_GCT_USB4125-xx-x-0190_6P_TopMnt_Horizontal.step"
 			(offset
 				(xyz 0 0 0)
@@
 			)
 			(rotate
-				(xyz 0 0 0)
+				(xyz -0 -0 -0)
 			)
 		)
@@
 		)
 		(embedded_fonts no)
-		(model "kicad-embed://dsgp_1575_18_4_a_02.obj"
+		(model "${KIPRJMOD}/libraries/DSGP.1575.18.4.A.02/dsgp_1575_18_4_a_02.stp"
 			(offset
 				(xyz 0 0 0)
@@
 			)
 			(rotate
-				(xyz 0 0 0)
+				(xyz -90 -0 -0)
 			)
 		)
@@
 	)
 	(via
+		(at 93.614317 93.3)
+		(size 0.6)
+		(drill 0.3)
+		(layers "F.Cu" "B.Cu")
+		(net "GND")
+	)
+	(via
 		(at 99.314317 86.5)
 		(size 0.6)
@@
 	)
 	(via
+		(at 91.014317 97.6)
+		(size 0.6)
+		(drill 0.3)
+		(layers "F.Cu" "B.Cu")
+		(net "GND")
+	)
+	(via
 		(at 127.314317 85.5)
 		(size 0.6)
@@
 	)
 	(via
+		(at 93.614317 94.3)
+		(size 0.6)
+		(drill 0.3)
+		(layers "F.Cu" "B.Cu")
+		(net "GND")
+	)
+	(via
 		(at 86.314317 72.5)
 		(size 0.6)
@@
 		(size 0.6)
 		(drill 0.3)
+		(layers "F.Cu" "B.Cu")
+		(net "GND")
+	)
+	(via
+		(at 92.014317 97.6)
+		(size 0.6)
+		(drill 0.3)
